File: SNES_CONTROLLER.kicad_pcb (KiCad board)
At the start: 2 copper layers, 57 x 76 mm, 24 parts, among them J1 Screw_Terminal_01x07, J2 Screw_Terminal_01x12, J3 Screw_Terminal_01x12, U1 4021, U2 4021

Commit message: SNES CONTROLLER v2
Parts:
- removed J1: Screw_Terminal_01x07, TerminalBlock:TerminalBlock_MaiXu_MX126-5.0-07P_1x07_P5.00mm
- added J4: Screw_Terminal_01x05, TerminalBlock:TerminalBlock_MaiXu_MX126-5.0-05P_1x05_P5.00mm, F.Cu at (116.2, 64.5)
Routing:
- net /Gnd: track 191.4 -> 0.00 mm
- net /Vcc: track 125.0 -> 120.2 mm
- net /Latch: track 82.6 -> 81.1 mm
- net /Clk: track 93.8 -> 92.3 mm
- net /Data1: track 87.5 -> 86.6 mm
- added copper zone on F.Cu, net /Gnd

Commit message: Error corrected. Pin 11 of second 4021 connected to GND
Connections:
- U2 pad 11: unconnected-(U2-DS-Pad11) -> /Gnd
Changed lines of the file:
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@@
 	(net 24 "Net-(U1-DS)")
 	(net 25 "unconnected-(U2-Q5-Pad2)")
-	(net 26 "unconnected-(U2-DS-Pad11)")
-	(net 27 "unconnected-(U2-Q6-Pad12)")
+	(net 26 "unconnected-(U2-Q6-Pad12)")
 	(footprint "Resistor_THT:R_Axial_DIN0207_L6.3mm_D2.5mm_P5.08mm_Vertical"
 		(layer "F.Cu")
@@
 			(layers "*.Cu" "*.Mask")
 			(remove_unused_layers no)
-			(net 26 "unconnected-(U2-DS-Pad11)")
+			(net 4 "/Gnd")
 			(pinfunction "DS")
-			(pintype "input+no_connect")
+			(pintype "input")
 		)
 		(pad "12" thru_hole oval
@@
 			(layers "*.Cu" "*.Mask")
 			(remove_unused_layers no)
-			(net 27 "unconnected-(U2-Q6-Pad12)")
+			(net 26 "unconnected-(U2-Q6-Pad12)")
 			(pinfunction "Q6")
 			(pintype "output+no_connect")
